File: Kicad/domus-silicea-raspberry-b.sch (KiCad schematic (older format))
At the start: 9 parts

Commit message: Step 31
Parts:
- removed D? (x2): IR333C LED, symbol LED
- removed Q? (x2): P2N2222AG, TO92-EBC, symbol BC237
- removed R?: 10K, symbol R
- removed R?: 560, symbol R
- removed U?: TSOP4838, symbol TSOP4838
- added D?: IR333C LED, symbol LED
- added Q? (x2): P2N2222AG, TO92-EBC, symbol BC237
- added R?: 10K, symbol R
- added R?: 560, symbol R
- added U?: TSOP4838, symbol TSOP4838
Connections:
- net +3.3V: now also D?.1 (A), R?.1, U?.3 (Vs)
- net GND: now also P?.9 (GND), Q?.E, Q?.E, R?.2, U?.2 (GND); no longer P?.6 (GND)
- net at P?.11 (GPIO17): now also Q?.B, Q?.B, R?.1
- net at P?.7 (GPIO4): now also U?.1 (OUT)
- net at P?.1 (In): now also Q?.C, R?.2
- net +5V: no longer names the net of P?.2 (5V)
- new net: D?.2 (K), Q?.C
Other:
- moved on the sheet: P?
