File: Eagle/prj/domus-silicea-board01-schematic.sch (EAGLE design)
At the start: 20 parts, among them CON1 POWER, CON2 REED, M1 ARDUINO-PRO-MINI-3.3V, M2 WIRELESS-NRF24L01, M3 WIRELESS-WIFI-ESP-01, M4 MOTION-PIR-HC-SR501, M5 TSOP38238, M6 DHT, Q1 BC487

Commit message: Eagle New Path
Parts:
- added PAD1, PAD2, PAD3, PAD4, PAD5, PAD6, PAD7: (no value), wirepad:2,54/1,0
- added PAD8: D3, wirepad:2,54/1,0
- added R6: 330, resistor:R-EU_0207/10
- added SJ3: +3V3, jumper:SJ
- added SJ4: +5V, jumper:SJ
- CON1: device pinhead:PINHD-1X2 -> pinhead:PINHD-1X3
- SJ1: value (none) -> PIR_H
- SJ2: value (none) -> PIR_L
Connections:
- new net +5V: CON1.1, M1.RAW, M4.VDD, PAD1.P, SJ4.2
- new net A0: M1.A0, PAD4.P
- new net A1: M1.A1, PAD5.P
- new net A2: M1.A2, PAD6.P
- new net A3: M1.A3, PAD7.P
- new net D3: M1.D3, PAD8.P
- new net LED: M1.D4, R6.2
- new net N$6: LED1.A, R6.1
- net +3V3: now also CON1.2, PAD2.P, SJ3.2; no longer C1.+, CON1.1
- net GND: now also CON1.3, LED1.C, PAD3.P; no longer CON1.2, M1.GND.3
- net N$4: now also C1.+, SJ3.1, SJ4.1; no longer CON2.1, R5.2
- net REED: now also CON2.1, R5.2
Other:
- moved on the sheet: C1, CON2, LED1, M3, R5
