File: Eagle/prj/domus-silicea-board02-schematic.sch (EAGLE design)
At the start: 33 parts, among them CON2 REED, M1 ARDUINO-PRO-MINI-3.3V, M2 WIRELESS-NRF24L01, M3 WIRELESS-WIFI-ESP-01, M4 MOTION-PIR-HC-SR501, M5 TSOP38238, M6 DHT, Q1 BC487, X1 POWER, X2 87758-0816

Commit message: Eagle_Board
Parts:
- added JP1, JP2: (no value), pinhead:PINHD-1X18
Changed lines of the file:
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@@
 <setting verticaltext="up"/>
 </settings>
-<grid distance="0.1" unitdist="inch" unit="inch" style="dots" multiple="1" display="no" altdistance="0.01" altunitdist="inch" altunit="inch"/>
+<grid distance="0.1" unitdist="inch" unit="inch" style="lines" multiple="1" display="no" altdistance="0.01" altunitdist="inch" altunit="inch"/>
 <layers>
 <layer number="1" name="Top" color="4" fill="1" visible="no" active="no"/>
@@
 </part>
 <part name="X2" library="con-molex" deviceset="87758-0816" device=""/>
+<part name="JP1" library="pinhead" deviceset="PINHD-1X18" device=""/>
+<part name="JP2" library="pinhead" deviceset="PINHD-1X18" device=""/>
 </parts>
 <sheets>
@@
 <instance part="X2" gate="-7" x="-10.16" y="15.24"/>
 <instance part="X2" gate="-8" x="10.16" y="15.24"/>
+<instance part="JP1" gate="A" x="147.32" y="78.74"/>
+<instance part="JP2" gate="A" x="160.02" y="78.74"/>
 </instances>
 <busses>
