File: Eagle/prj/domus-silicea-board03-schematic.sch (EAGLE design)
At the start: 35 parts, among them CON2 REED, M1 ARDUINO-PRO-MINI-3.3V, M2 WIRELESS-NRF24L01, M3 WIRELESS-WIFI-ESP-01, M4 MOTION-PIR-HC-SR501, M5 TSOP38238, M6 DHT, Q1 BC487, X1 POWER, X2 87758-0816

Commit message: domus-silicea - M1 - Arduino Pro-Mini
Parts:
- removed D1: 1N4004, diode:1N4004
- removed PAD1, PAD2, PAD3, PAD4, PAD5, PAD6, PAD7: (no value), wirepad:2,54/1,0
- removed PAD8: D3, wirepad:2,54/1,0
- removed X2: 87758-0816, con-molex:87758-0816
- added JP3, JP4: (no value), pinhead:PINHD-1X6
- C1: value (none) -> 10uF
- JP1, JP2: device pinhead:PINHD-1X18 -> pinhead:PINHD-1X6
Connections:
- removed net +3V3: M1.VCC, M2.VCC, M3.CH_PD, M3.VCC, M4.+3V3, M5.VCC, M6.VCC, PAD2.P, R2.2, R3.2, R4.1, R5.1, SJ1.1, SJ3.2, X1-2.S
- removed net +5V: M1.RAW, M4.VDD, PAD1.P, SJ4.2, X1-1.S
- removed net DHT: M1.D8, M6.OUT, R4.2
- removed net ESP_RX: M1.D1/TX, M3.URXD
- removed net ESP_TX: M1.D0/RX, M3.UTXD
- removed net IR_RX: M1.D7, M5.OUT
- removed net IR_TX: M1.D6, R1.1
- removed net LED: M1.D4, R6.2
- removed net N24_CE: M1.D9, M2.CE
- removed net N24_CSN: M1.D10, M2.CSN
- removed net N24_MISO: M1.D12, M2.MISO
- removed net N24_MOSI: M1.D11, M2.MOSI
- removed net N24_SCK: M1.D13, M2.SCK
- removed net PIR: M1.D2, M4.OUT, R3.1
- removed net REED: CON2.1, M1.D5, R5.2
- new net D0/RX: JP1.2, M1.D0/RX, M3.UTXD
- new net D1/TX: JP1.1, M1.D1/TX, M3.URXD
- new net D10: JP4.6, M1.D10, M2.CSN
- new net D11: JP4.5, M1.D11, M2.MOSI
- new net D12: JP4.4, M1.D12, M2.MISO
- new net D13: JP4.3, M1.D13, M2.SCK
- new net D2: JP1.5, M1.D2, M4.OUT, R3.1
- new net D4: JP2.1, M1.D4, R6.2
- new net D5: CON2.1, JP2.2, M1.D5, R5.2
- new net D6: JP2.3, M1.D6, R1.1
- new net D7: JP2.4, M1.D7, M5.OUT
- new net D8: JP2.5, M1.D8, M6.OUT, R4.2
- new net D9: JP2.6, M1.D9, M2.CE
- new net RAW: JP3.1, M1.RAW, M4.VDD, SJ4.2, X1-1.S
- new net RST: JP1.3, JP3.3, M1.RST.1, M1.RST.2
- new net VCC: JP3.4, M1.VCC, M2.VCC, M3.CH_PD, M3.VCC, M4.+3V3, M5.VCC, M6.VCC, R2.2, R3.2, R4.1, R5.1, SJ1.1, SJ3.2, X1-2.S
- net A0: now also JP4.2; no longer PAD4.P
- net A1: now also JP4.1; no longer PAD5.P
- net A2: now also JP3.6; no longer PAD6.P
- net A3: now also JP3.5; no longer PAD7.P
- net D3: now also JP1.6; no longer PAD8.P
- net GND: now also JP1.4, JP3.2; no longer PAD3.P
Other:
- moved on the sheet: C1, M1, M2, M3, SJ3, SJ4, X1-1, X1-2, X1-3
