File: Eagle/prj/domus-silicea - N2 - ESP8266-01.sch (EAGLE design)
At the start: 27 parts, among them CON2 REED, M1 ARDUINO-PRO-MINI-3.3V, M2 WIRELESS-NRF24L01, M3 WIRELESS-WIFI-ESP-01, M4 MOTION-PIR-HC-SR501, M5 TSOP38238, M6 DHT, Q1 BC487, X1 POWER

Commit message: EASYIOT_OLED
Parts:
- removed C1, C2: 10uF, rcl:CPOL-EUE2,5-6E
- removed CON2: REED, pinhead:PINHD-1X2
- removed IRLED1, IRLED2, LED1: (no value), led:LED5MM
- removed M1: ARDUINO-PRO-MINI-3.3V, diy-modules:ARDUINO-PRO-MINI-3.3V
- removed M2: WIRELESS-NRF24L01, diy-modules:WIRELESS-NRF24L01
- removed M4: MOTION-PIR-HC-SR501, domus-silicea:MOTION-PIR-HC-SR501
- removed M5: TSOP38238, domus-silicea:TSOP38238
- removed M6: DHT, domus-silicea:DHT
- removed Q1: BC487, transistor-npn:BC487
- removed R1: 220, resistor:R-US_0204/7
- removed R2: 0, resistor:R-US_0204/7
- removed R3, R4: 10K, resistor:R-US_0204/7
- removed R5: 1M, resistor:R-US_0204/7
- removed R6: 330, resistor:R-US_0204/7
- removed SJ1: PIR_H, jumper:SJ
- removed SJ2: PIR_L, jumper:SJ
- removed SJ3: +3V3, jumper:SJ
- removed SJ4: +5V, jumper:SJ
- removed X1: POWER, con-molex:22-23-2031
- C3: value 10uF -> (none)
Connections:
- removed net N$1: IRLED1.C, IRLED2.C, Q1.C
- removed net N$2: IRLED1.A, IRLED2.A, R2.1
- removed net N$3: Q1.B, R1.2
- removed net N$4: C1.+, SJ3.1, SJ4.1
- removed net N$5: M4.TRG, SJ1.2, SJ2.2
- removed net N$6: LED1.A, R6.1
- net A0: no longer M1.A0
- net A1: no longer M1.A1
- net A2: no longer M1.A2
- net A3: no longer M1.A3
- net D0/RX: no longer M1.D0/RX
- net D1/TX: no longer M1.D1/TX
- net D10: no longer M1.D10, M2.CSN
- net D11: no longer M1.D11, M2.MOSI
- net D12: no longer M1.D12, M2.MISO
- net D13: no longer M1.D13, M2.SCK
- net D2: no longer M1.D2, M4.OUT, R3.1
- net D3: no longer M1.D3
- net D4: no longer M1.D4, R6.2
- net D5: no longer CON2.1, M1.D5, R5.2
- net D6: no longer M1.D6, R1.1
- net D7: no longer M1.D7, M5.OUT
- net D8: no longer M1.D8, M6.OUT, R4.2
- net D9: no longer M1.D9, M2.CE
- net GND: no longer C1.-, C2.-, CON2.2, LED1.C, M1.GND.1, M1.GND.2, M2.GND, M4.GND.1, M4.GND.2, M5.GND, M6.GND, Q1.E, SJ2.1, X1-3.S
- net RAW: no longer M1.RAW, M4.VDD, SJ4.2, X1-1.S
- net RST: no longer M1.RST.1, M1.RST.2
- net VCC: no longer C2.+, M1.VCC, M2.VCC, M4.+3V3, M5.VCC, M6.VCC, R2.2, R3.2, R4.1, R5.1, SJ1.1, SJ3.2, X1-2.S
Other:
- moved on the sheet: C3, JP1, JP2, M3
